File: Electrónica/propuesta1/propuesta1.kicad_sch (KiCad schematic)
At the start: 69 parts, among them K1 SANYOU_SRD_Form_C, M1 Trituradora_motor, M2 Fan, M3 Fan, M4 NEMA17, M5 NEMA17, Q1 2N2222A-TO92, Q2 BTA12-600B, Q3 BTA12-600B, Q4 BTA12-600B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

Commit message: modified:   pcb
Parts:
- removed TC1, TC2, TC3: Thermocouple_Block, symbol Device:Thermocouple_Block
- removed U3, U4: AS5045B, 4ms_Encoder:ENC_SPST_12mm, symbol Sensor_Magnetic:AS5045B
- added C11, C12, C13: 100nf, PCM_Capacitor_THT_AKL:C_Disc_D4.7mm_W2.5mm_P5.00mm, symbol Device:C_Small
- added J1: Funete conmutada, symbol Connector:Screw_Terminal_01x02
- added J4, J5, J6: Max6675_modulo, Connector_PinHeader_2.54mm:PinHeader_1x05_P2.54mm_Horizontal, symbol Connector:Conn_01x05_Pin
- added J7: ESP01, Connector_PinHeader_2.54mm:PinHeader_1x04_P2.54mm_Horizontal, symbol Connector:Conn_01x04_Pin
- added R25: 1k, PCM_Resistor_THT_AKL:R_Axial_DIN0207_L6.3mm_D2.5mm_P10.16mm_Horizontal, symbol Device:R_US
- added R26: 2k, PCM_Resistor_THT_AKL:R_Axial_DIN0207_L6.3mm_D2.5mm_P10.16mm_Horizontal, symbol Device:R_US
- added U3: LM7805CT, PCM_Package_TO_SOT_THT_AKL:TO-220-3_Vertical, symbol PCM_Voltage_Regulator_AKL:LM7805CT
- added U5: 74HC14, symbol 74xx:74HC14
- added U6: ESP-01S, RF_Module:ESP-01, symbol speedy_hardware_items:ESP-01s
- C10: footprint (none) -> PCM_Capacitor_THT_AKL:C_Disc_D4.7mm_W2.5mm_P5.00mm
- C4, C6, C8: value 0.1uf -> 0.1uf poliester
- R1, R10, R11, R13, R14, R15, R17, R18, R19, R4, R5, R6, R8, R9, RV1, RV2: footprint (none) -> PCM_Resistor_THT_AKL:R_Axial_DIN0207_L6.3mm_D2.5mm_P10.16mm_Horizontal
- R12, R16, R20: footprint (none) -> PCM_Resistor_THT_AKL:R_Axial_DIN0411_L9.9mm_D3.6mm_P15.24mm_Horizontal
- R22: value 180 -> 10k; footprint (none) -> PCM_Resistor_THT_AKL:R_Axial_DIN0207_L6.3mm_D2.5mm_P10.16mm_Horizontal
- R23, R24: value 47K 1W -> 5K 2W; footprint (none) -> PCM_Resistor_THT_AKL:R_Axial_DIN0414_L11.9mm_D4.5mm_P15.24mm_Horizontal
Connections:
- net 127VAC: no longer R23.1
- net 12VCC_nema: now also J1.2 (Pin_2), U3.1 (IN)
- net 5VCC: now also C11.2, C12.2, C13.2, U5.14 (VCC)
- net Calfactor0: now also U5.3; no longer R8.2
- net Calfactor1: now also U5.5, U5.9; no longer R13.2, R17.2
- net GND2: now also C11.1, C12.1, C13.1, J1.1 (Pin_1), R26.2, U3.2, U5.7 (GND)
- net NEUT: now also R23.1; no longer D4.2 (1)
- net at D4.4 (2), R24.2: no longer R23.2
- net at OC4.4, R22.2: now also U5.1
- new net: R17.2, U5.8
- new net: R25.1, U5.2
- new net: D4.2 (1), R23.2
- new net: R8.2, U5.4
- new net: R13.2, U5.6
- new net +3.3V: J7.1 (Pin_1), U6.7 (VCC)
- new net +5V: J4.2 (Pin_2), J5.2 (Pin_2), J6.2 (Pin_2)
- new net GND: J4.1 (Pin_1), J5.1 (Pin_1), J6.1 (Pin_1), J7.4 (Pin_4), U6.2 (GND)
- new net Rx_mcu_esp01: J7.2 (Pin_2), U6.1 (TX)
- new net Tx_mcu_esp01: J7.3 (Pin_3), U6.8 (RX)
- new net cs0: J4.4 (Pin_4)
- new net cs1: J5.4 (Pin_4)
- new net cs2: J6.4 (Pin_4)
- new net sck: J4.3 (Pin_3), J5.3 (Pin_3), J6.3 (Pin_3)
- new net so: J4.5 (Pin_5), J5.5 (Pin_5), J6.5 (Pin_5)
- new net zc: R25.2, R26.1
- no-connect marks 31 -> 35
Other:
- note added: "Alimentación"
- note added: "Control"
- note added: "Cruce por cero"
- moved on the sheet: C10, C4, C5, C6, C7, C8, C9, D4, M2, M3, OC1, OC2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

Commit message: new file:   "Electr\303\263nica/propuesta1/propuesta1-backups/propuesta1-2025-04-02_221845.zip" 	new file:   "Electr\303\263nica/propuesta1/propuesta1-backups/propuesta1-2025-04-02_222917.zip" 	new file:   "Electr\303\263nica/propuesta1/propuesta1-backups/propuesta1-2025-04-02_230044.zip" 	modified:   "Electr\303\263nica/propuesta1/propuesta1.kicad_sch" 	new file:   "Investigaci\303\263n_fuentes/siov-applications.pdf"
Parts:
- added F2, F3, F4: 2A, symbol Device:Fuse
- added F5: 0.5, symbol Device:Fuse
- added R27, R28, R29: 10k, PCM_Resistor_THT_AKL:R_Axial_DIN0207_L6.3mm_D2.5mm_P10.16mm_Horizontal, symbol Device:R_US
- added RV3, RV4, RV5, RV6: 10D241K 240V, Varistor:RV_Disc_D7mm_W3.4mm_P5mm, symbol Device:Varistor_US
- R21, R3, R7: value Heater -> Heater 100W
Connections:
- net 127VAC: now also F2.2, F3.2, F4.2, F5.2; no longer R21.2, R24.1, R3.2, R7.2
- net 5VCC: now also R27.1, R28.1, R29.1
- net Calfactor0: now also R29.2
- net Calfactor1: now also R27.2, R28.2
- net NEUT: now also RV3.2, RV4.2, RV5.2, RV6.2
- new net: F2.1, R3.2, RV3.1
- new net: F5.1, R24.1, RV6.1
- new net: F4.1, R21.2, RV5.1
- new net: F3.1, R7.2, RV4.1
Other:
- moved on the sheet: R21, R3, R7
